Commit message: made first joint and link in xacro made .rviz file for xacro made launch file for xacro testing

File: diff_drive/urdf/ddrive.urdf.xacro (robot description, xacro)
@@ -4,5 +4,29 @@
 <xacro:property name='dimyaml' value='$(find diff_drive)/config/dims.yaml'/>
 <xacro:property name='dims' value='${load_yaml(dimyaml)}'/>
-<xacro:property name='L' value='${dims["L"]}' />
-<xacro:property name='W' value='${dims["W"]}' />
-<xacro:property name='H' value='${dims["H"]}' />
+<xacro:property name='L' value='${dims["L"]}'/>
+<xacro:property name='W' value='${dims["W"]}'/>
+<xacro:property name='H' value='${dims["H"]}'/>
+<link name='base_footprint' type='fixed'/>
+<joint name='base_joint' type='fixed'>
+    <parent link='base_footprint'/>
+    <child link='base_link'/>
+    <origin xyz='0 0 0' rpy='0 0 0'/>
+</joint>
+<link name='base_link'>
+    <visual>
+        <origin xyz='0 0 ${H/2}'/>
+        <geometry>
+            <box size='${L} ${W} ${H}'/>
+        </geometry>
+        <material name='green_mat'>
+            <color rgba='0 1 0 1' />
+        </material>
+    </visual>
+    <collision>
+        <origin xyz='0 0 ${H/2}'/>
+        <geometry>
+            <box size='${L} ${W} ${H}'/>
+        </geometry>
+    </collision>
+</link>
+</robot>

Commit message: xacro as both back wheels

File: diff_drive/urdf/ddrive.urdf.xacro (robot description, xacro)
@@ -1,32 +1,95 @@
 <?xml version="1.0"?>
 <robot xmlns:xacro="http://www.ros.org/wiki/xacro" name="cybercaster">
-<!-- Load from yaml file -->
-<xacro:property name='dimyaml' value='$(find diff_drive)/config/dims.yaml'/>
-<xacro:property name='dims' value='${load_yaml(dimyaml)}'/>
-<xacro:property name='L' value='${dims["L"]}'/>
-<xacro:property name='W' value='${dims["W"]}'/>
-<xacro:property name='H' value='${dims["H"]}'/>
-<link name='base_footprint' type='fixed'/>
-<joint name='base_joint' type='fixed'>
-    <parent link='base_footprint'/>
-    <child link='base_link'/>
-    <origin xyz='0 0 0' rpy='0 0 0'/>
-</joint>
-<link name='base_link'>
-    <visual>
-        <origin xyz='0 0 ${H/2}'/>
-        <geometry>
-            <box size='${L} ${W} ${H}'/>
-        </geometry>
-        <material name='green_mat'>
-            <color rgba='0 1 0 1' />
-        </material>
-    </visual>
-    <collision>
-        <origin xyz='0 0 ${H/2}'/>
-        <geometry>
-            <box size='${L} ${W} ${H}'/>
-        </geometry>
-    </collision>
-</link>
+    <!-- Load from yaml file -->
+    <xacro:property name='dimyaml' value='$(find diff_drive)/config/dims.yaml'/>
+    <xacro:property name='dims' value='${load_yaml(dimyaml)}'/>
+    <xacro:property name='L' value='${dims["L"]}'/>
+    <xacro:property name='W' value='${dims["W"]}'/>
+    <xacro:property name='H' value='${dims["H"]}'/>
+    <xacro:property name='R' value='${H}'/>
+    <xacro:property name='WL' value='${W/5}'/>
+    <link name='base_footprint' type='fixed'/>
+    <joint name='base_joint' type='fixed'>
+        <parent link='base_footprint'/>
+        <child link='base_link'/>
+        <origin xyz='0 0 0' rpy='0 0 0'/>
+    </joint>
+    <link name='base_link'>
+        <visual>
+            <origin xyz='0 0 ${H/2}'/>
+            <geometry>
+                <box size='${L} ${W} ${H}'/>
+            </geometry>
+            <material name='cyan_mat'>
+                <color rgba='0 1 1 1' />
+            </material>
+        </visual>
+        <collision>
+            <origin xyz='0 0 ${H/2}'/>
+            <geometry>
+                <box size='${L} ${W} ${H}'/>
+            </geometry>
+        </collision>
+        <inertial>
+            <origin xyz='0 0 ${H/2}'/>
+            <mass value='0.5'/>
+            <inertia ixx="${(L+W**3)/12}" ixy="0" ixz="0"
+               iyy="${(W+L**3)/12}" iyz="0"
+               izz="${(L*W*(L**2+W**2))/12}" />
+        </inertial>
+    </link>
+    <joint name="left_wheel" type='continuous'>
+        <parent link="base_link"/>
+        <child link="left_wheel_link"/>
+        <origin xyz="${L/4} ${-W/2-WL/2} ${H/2}" rpy='${-pi/2} 0 0'/>
+        <axis xyz="0 1 0"/>
+    </joint>
+    <link name="left_wheel_link">
+        <visual>
+            <geometry>
+                <cylinder radius='${R}' length='${WL}'/>
+            </geometry>
+            <material name="pink_mat">
+                <color rgba='1 0 1 1'/>
+            </material>
+        </visual>
+        <collision>
+            <geometry>
+                <cylinder length='${R}' radius='${WL}'/>
+            </geometry>
+        </collision>
+        <inertial>
+            <mass value="0.1" />
+            <inertia ixx="${(pi*R**4)/4}" ixy="0" ixz="0"
+                iyy="${(pi*R**4)/4}" iyz="0"
+                izz="${(pi*R**4)/2}" />
+        </inertial>
+    </link>
+    <joint name="right_wheel" type='continuous'>
+        <parent link="base_link"/>
+        <child link="right_wheel_link"/>
+        <origin xyz="${L/4} ${W/2+WL/2} ${H/2}" rpy='${-pi/2} 0 0'/>
+        <axis xyz="0 1 0"/>
+    </joint>
+    <link name="right_wheel_link">
+        <visual>
+            <geometry>
+                <cylinder radius='${R}' length='${WL}'/>
+            </geometry>
+            <material name="pink_mat">
+                <color rgba='1 0 1 1'/>
+            </material>
+        </visual>
+        <collision>
+            <geometry>
+                <cylinder length='${R}' radius='${WL}'/>
+            </geometry>
+        </collision>
+        <inertial>
+            <mass value="0.1" />
+            <inertia ixx="${(pi*R**4)/4}" ixy="0" ixz="0"
+                iyy="${(pi*R**4)/4}" iyz="0"
+                izz="${(pi*R**4)/2}" />
+        </inertial>
+    </link>
 </robot>

Commit message: finished first iteration of xacro

File: diff_drive/urdf/ddrive.urdf.xacro (robot description, xacro)
@@ -43,5 +43,5 @@
         <child link="left_wheel_link"/>
         <origin xyz="${L/4} ${-W/2-WL/2} ${H/2}" rpy='${-pi/2} 0 0'/>
-        <axis xyz="0 1 0"/>
+        <axis xyz="0 0 1"/>
     </joint>
     <link name="left_wheel_link">
@@ -70,5 +70,5 @@
         <child link="right_wheel_link"/>
         <origin xyz="${L/4} ${W/2+WL/2} ${H/2}" rpy='${-pi/2} 0 0'/>
-        <axis xyz="0 1 0"/>
+        <axis xyz="0 0 1"/>
     </joint>
     <link name="right_wheel_link">
@@ -93,3 +93,55 @@
         </inertial>
     </link>
+    <joint name="caster_bottom_joint" type="fixed">
+        <parent link="base_link"/>
+        <child link="caster_bottom_link"/>
+        <origin xyz="${-3*L/8} 0 0" rpy="${-pi/2} 0 0"/>
+    </joint>
+    <link name="caster_bottom_link">
+        <visual>
+            <geometry>
+                <sphere radius='${R-(H/2)}'/>
+            </geometry>
+            <material name="yellow_mat">
+                <color rgba='1 1 0 1'/>
+            </material>
+        </visual>
+        <collision>
+            <geometry>
+                <sphere radius='${R-(H/2)}'/>
+            </geometry>
+        </collision>
+        <inertial>
+            <mass value="0.1" />
+            <inertia ixx="${(2/5)*0.1*(R-(H/2))**2}" ixy="0.0" ixz="0.0"
+                iyy="${(2/5)*0.1*(R-(H/2))**2}" iyz="0.0"
+                izz="${(2/5)*0.1*(R-(H/2))**2}" />
+        </inertial>
+    </link>
+    <joint name="caster_top_joint" type="fixed">
+        <parent link="base_link"/>
+        <child link="caster_top_link"/>
+        <origin xyz="${-3*L/8} 0 ${H}" rpy="${-pi/2} 0 0"/>
+    </joint>
+    <link name="caster_top_link">
+        <visual>
+            <geometry>
+                <sphere radius='${R-(H/2)}'/>
+            </geometry>
+            <material name="yellow_mat">
+                <color rgba='1 1 0 1'/>
+            </material>
+        </visual>
+        <collision>
+            <geometry>
+                <sphere radius='${R-(H/2)}'/>
+            </geometry>
+        </collision>
+        <inertial>
+            <mass value="0.1" />
+            <inertia ixx="${(2/5)*0.1*(R-(H/2))**2}" ixy="0.0" ixz="0.0"
+                iyy="${(2/5)*0.1*(R-(H/2))**2}" iyz="0.0"
+                izz="${(2/5)*0.1*(R-(H/2))**2}" />
+        </inertial>
+    </link>
 </robot>

Commit message: fixed inertia values

File: diff_drive/urdf/ddrive.urdf.xacro (robot description, xacro)
@@ -9,4 +9,6 @@
     <xacro:property name='R' value='${H}'/>
     <xacro:property name='WL' value='${W/5}'/>
+    <xacro:property name='MR' value='0.5'/>
+    <xacro:property name='MW' value='0.1'/>
     <link name='base_footprint' type='fixed'/>
     <joint name='base_joint' type='fixed'>
@@ -17,5 +19,5 @@
     <link name='base_link'>
         <visual>
-            <origin xyz='0 0 ${H/2}'/>
+            <origin xyz='0 0 0'/>
             <geometry>
                 <box size='${L} ${W} ${H}'/>
@@ -33,8 +35,8 @@
         <inertial>
             <origin xyz='0 0 ${H/2}'/>
-            <mass value='0.5'/>
-            <inertia ixx="${(L+W**3)/12}" ixy="0" ixz="0"
-               iyy="${(W+L**3)/12}" iyz="0"
-               izz="${(L*W*(L**2+W**2))/12}" />
+            <mass value='${MR}'/>
+            <inertia ixx="${MR*(H**2+W**2)/12}" ixy="0" ixz="0"
+               iyy="${MR*(H**2+L**2)/12}" iyz="0"
+               izz="${MR*(L**2+W**2)/12}" />
         </inertial>
     </link>
@@ -42,5 +44,5 @@
         <parent link="base_link"/>
         <child link="left_wheel_link"/>
-        <origin xyz="${L/4} ${-W/2-WL/2} ${H/2}" rpy='${-pi/2} 0 0'/>
+        <origin xyz="${L/4} ${-W/2-WL/2} 0" rpy='${-pi/2} 0 0'/>
         <axis xyz="0 0 1"/>
     </joint>
@@ -56,12 +58,12 @@
         <collision>
             <geometry>
-                <cylinder length='${R}' radius='${WL}'/>
+                <cylinder radius='${R}' length='${WL}'/>
             </geometry>
         </collision>
         <inertial>
-            <mass value="0.1" />
-            <inertia ixx="${(pi*R**4)/4}" ixy="0" ixz="0"
-                iyy="${(pi*R**4)/4}" iyz="0"
-                izz="${(pi*R**4)/2}" />
+            <mass value="${MW}" />
+            <inertia ixx="${(1/12)*MW*(3*R**2+WL**2)}" ixy="0" ixz="0"
+                iyy="${(1/12)*MW*(3*R**2+WL**2)}" iyz="0"
+                izz="${0.5*MW*R**2}" />
         </inertial>
     </link>
@@ -69,5 +71,5 @@
         <parent link="base_link"/>
         <child link="right_wheel_link"/>
-        <origin xyz="${L/4} ${W/2+WL/2} ${H/2}" rpy='${-pi/2} 0 0'/>
+        <origin xyz="${L/4} ${W/2+WL/2} 0" rpy='${-pi/2} 0 0'/>
         <axis xyz="0 0 1"/>
     </joint>
@@ -83,12 +85,12 @@
         <collision>
             <geometry>
-                <cylinder length='${R}' radius='${WL}'/>
+                <cylinder radius='${R}' length='${WL}'/>
             </geometry>
         </collision>
         <inertial>
             <mass value="0.1" />
-            <inertia ixx="${(pi*R**4)/4}" ixy="0" ixz="0"
-                iyy="${(pi*R**4)/4}" iyz="0"
-                izz="${(pi*R**4)/2}" />
+            <inertia ixx="${(1/12)*MW*(3*R**2+WL**2)}" ixy="0" ixz="0"
+                iyy="${(1/12)*MW*(3*R**2+WL**2)}" iyz="0"
+                izz="${0.5*MW*R**2}" />
         </inertial>
     </link>
@@ -96,5 +98,5 @@
         <parent link="base_link"/>
         <child link="caster_bottom_link"/>
-        <origin xyz="${-3*L/8} 0 0" rpy="${-pi/2} 0 0"/>
+        <origin xyz="${-3*L/8} 0 ${-H/2}" rpy="${-pi/2} 0 0"/>
     </joint>
     <link name="caster_bottom_link">
@@ -113,8 +115,8 @@
         </collision>
         <inertial>
-            <mass value="0.1" />
-            <inertia ixx="${(2/5)*0.1*(R-(H/2))**2}" ixy="0.0" ixz="0.0"
-                iyy="${(2/5)*0.1*(R-(H/2))**2}" iyz="0.0"
-                izz="${(2/5)*0.1*(R-(H/2))**2}" />
+            <mass value="${MW}" />
+            <inertia ixx="${(2/5)*MW*(R-(H/2))**2}" ixy="0.0" ixz="0.0"
+                iyy="${(2/5)*MW*(R-(H/2))**2}" iyz="0.0"
+                izz="${(2/5)*MW*(R-(H/2))**2}" />
         </inertial>
     </link>
@@ -122,5 +124,5 @@
         <parent link="base_link"/>
         <child link="caster_top_link"/>
-        <origin xyz="${-3*L/8} 0 ${H}" rpy="${-pi/2} 0 0"/>
+        <origin xyz="${-3*L/8} 0 ${H/2}" rpy="${-pi/2} 0 0"/>
     </joint>
     <link name="caster_top_link">
@@ -139,8 +141,8 @@
         </collision>
         <inertial>
-            <mass value="0.1" />
-            <inertia ixx="${(2/5)*0.1*(R-(H/2))**2}" ixy="0.0" ixz="0.0"
-                iyy="${(2/5)*0.1*(R-(H/2))**2}" iyz="0.0"
-                izz="${(2/5)*0.1*(R-(H/2))**2}" />
+            <mass value="${MW}" />
+            <inertia ixx="${(2/5)*MW*(R-(H/2))**2}" ixy="0.0" ixz="0.0"
+                iyy="${(2/5)*MW*(R-(H/2))**2}" iyz="0.0"
+                izz="${(2/5)*MW*(R-(H/2))**2}" />
         </inertial>
     </link>

Commit message: flips are good to go need to fix follow_rect need to clean code

File: diff_drive/urdf/ddrive.urdf.xacro (robot description, xacro)
@@ -18,7 +18,7 @@
     <!-- <xacro:property name='MC' value='0.5'/> -->
     <!-- default for masses for rect -->
-    <xacro:property name='MR' value='0.1'/>
+    <xacro:property name='MR' value='0.01'/>
     <!-- <xacro:property name='MW' value='0.02'/> -->
-    <xacro:property name='MC' value='0.02'/>
+    <xacro:property name='MC' value='0.01'/>
     <link name='base_footprint' type='fixed'/>
     <joint name='base_joint' type='fixed'>
