Commit message: xacro successfully imported to Gazebo with usable physics and material qualities

File: diff_drive/urdf/ddrive.gazebo.xacro (robot description, xacro)
@@ -22,5 +22,5 @@
         <maxVel>0.1</maxVel>
         <fdir1>1 0 0</fdir1>
-        <material>Gazebo/FlatBlack</material>
+        <material>Gazebo/PurpleGlow</material>
     </gazebo>
     <gazebo reference="right_wheel_link">
@@ -32,5 +32,5 @@
         <maxVel>0.1</maxVel>
         <fdir1>1 0 0</fdir1>
-        <material>Gazebo/FlatBlack</material>
+        <material>Gazebo/PurpleGlow</material>
     </gazebo>
     <gazebo reference="caster_bottom_link">
@@ -40,6 +40,6 @@
         <kd>100.0</kd>
         <minDepth>0.001</minDepth>
-        <maxVel>1.0</maxVel>
-        <material>Gazebo/FlatBlack</material>
+        <maxVel>1</maxVel>
+        <material>Gazebo/YellowGlow</material>
     </gazebo>
     <gazebo reference="caster_top_link">
@@ -49,6 +49,6 @@
         <kd>100.0</kd>
         <minDepth>0.001</minDepth>
-        <maxVel>1.0</maxVel>
-        <material>Gazebo/FlatBlack</material>
+        <maxVel>1</maxVel>
+        <material>Gazebo/YellowGlow</material>
     </gazebo>
 </robot>

File: diff_drive/urdf/ddrive.urdf.xacro (robot description, xacro)
@@ -23,5 +23,4 @@
     <link name='base_link'>
         <visual>
-            <origin xyz='0 0 0'/>
             <geometry>
                 <box size='${L} ${W} ${H}'/>
@@ -32,5 +31,4 @@
         </visual>
         <collision>
-            <origin xyz='0 0 ${H/2}'/>
             <geometry>
                 <box size='${L} ${W} ${H}'/>
@@ -38,5 +36,4 @@
         </collision>
         <inertial>
-            <origin xyz='0 0 ${H/2}'/>
             <mass value='${MR}'/>
             <inertia ixx="${MR*(H**2+W**2)/12}" ixy="0" ixz="0"

Commit message: refined accuracy of trajectory following reduced robot mass for accuracy

File: diff_drive/urdf/ddrive.gazebo.xacro (robot description, xacro)
@@ -12,6 +12,6 @@
     <xacro:property name='WL' value='${W/5}'/>
     <!-- masses -->
-    <xacro:property name='MR' value='0.5'/>
-    <xacro:property name='MW' value='0.1'/>
+    <xacro:property name='MR' value='0.1'/>
+    <xacro:property name='MW' value='0.02'/>
     <gazebo reference="base_link">
         <material>Gazebo/TurquoiseGlow</material>

File: diff_drive/urdf/ddrive.urdf.xacro (robot description, xacro)
@@ -13,6 +13,6 @@
     <xacro:property name='WL' value='${W/5}'/>
     <!-- masses -->
-    <xacro:property name='MR' value='0.5'/>
-    <xacro:property name='MW' value='0.1'/>
+    <xacro:property name='MR' value='0.1'/>
+    <xacro:property name='MW' value='0.02'/>
     <link name='base_footprint' type='fixed'/>
     <joint name='base_joint' type='fixed'>

Commit message: best flips so far

File: diff_drive/urdf/ddrive.gazebo.xacro (robot description, xacro)
@@ -9,9 +9,7 @@
     <xacro:property name='H' value='${dims["H"]}'/>
     <!-- wheel radius and length -->
-    <xacro:property name='R' value='${H}'/>
+    <!-- <xacro:property name='R' value='${H}'/> -->
+    <xacro:property name='R' value='${1.25*H}'/>
     <xacro:property name='WL' value='${W/5}'/>
-    <!-- masses -->
-    <xacro:property name='MR' value='0.1'/>
-    <xacro:property name='MW' value='0.02'/>
     <gazebo reference="base_link">
         <material>Gazebo/TurquoiseGlow</material>

File: diff_drive/urdf/ddrive.urdf.xacro (robot description, xacro)
@@ -10,9 +10,15 @@
     <xacro:property name='H' value='${dims["H"]}'/>
     <!-- wheel radius and length -->
-    <xacro:property name='R' value='${H}'/>
+    <!-- <xacro:property name='R' value='${H}'/> -->
+    <xacro:property name='R' value='${1.25*H}'/>
     <xacro:property name='WL' value='${W/5}'/>
     <!-- masses -->
+    <!-- <xacro:property name='MR' value='1'/> -->
+    <xacro:property name='MW' value='0.5'/>
+    <!-- <xacro:property name='MC' value='0.5'/> -->
+    <!-- default for masses for rect -->
     <xacro:property name='MR' value='0.1'/>
-    <xacro:property name='MW' value='0.02'/>
+    <!-- <xacro:property name='MW' value='0.02'/> -->
+    <xacro:property name='MC' value='0.02'/>
     <link name='base_footprint' type='fixed'/>
     <joint name='base_joint' type='fixed'>
@@ -45,5 +51,5 @@
         <parent link="base_link"/>
         <child link="left_wheel_link"/>
-        <origin xyz="${L/4} ${-W/2-WL/2} 0" rpy='${-pi/2} 0 0'/>
+        <origin xyz="${L/2} ${-W/2-WL/2} 0" rpy='${-pi/2} 0 0'/>
         <axis xyz="0 0 1"/>
     </joint>
@@ -72,5 +78,5 @@
         <parent link="base_link"/>
         <child link="right_wheel_link"/>
-        <origin xyz="${L/4} ${W/2+WL/2} 0" rpy='${-pi/2} 0 0'/>
+        <origin xyz="${L/2} ${W/2+WL/2} 0" rpy='${-pi/2} 0 0'/>
         <axis xyz="0 0 1"/>
     </joint>
@@ -116,8 +122,8 @@
         </collision>
         <inertial>
-            <mass value="${MW}" />
-            <inertia ixx="${(2/5)*MW*(R-(H/2))**2}" ixy="0.0" ixz="0.0"
-                iyy="${(2/5)*MW*(R-(H/2))**2}" iyz="0.0"
-                izz="${(2/5)*MW*(R-(H/2))**2}" />
+            <mass value="${MC}" />
+            <inertia ixx="${(2/5)*MC*(R-(H/2))**2}" ixy="0.0" ixz="0.0"
+                iyy="${(2/5)*MC*(R-(H/2))**2}" iyz="0.0"
+                izz="${(2/5)*MC*(R-(H/2))**2}" />
         </inertial>
     </link>
@@ -142,8 +148,8 @@
         </collision>
         <inertial>
-            <mass value="${MW}" />
-            <inertia ixx="${(2/5)*MW*(R-(H/2))**2}" ixy="0.0" ixz="0.0"
-                iyy="${(2/5)*MW*(R-(H/2))**2}" iyz="0.0"
-                izz="${(2/5)*MW*(R-(H/2))**2}" />
+            <mass value="${MC}" />
+            <inertia ixx="${(2/5)*MC*(R-(H/2))**2}" ixy="0.0" ixz="0.0"
+                iyy="${(2/5)*MC*(R-(H/2))**2}" iyz="0.0"
+                izz="${(2/5)*MC*(R-(H/2))**2}" />
         </inertial>
     </link>

Commit message: cleaned code commented code

File: diff_drive/urdf/ddrive.gazebo.xacro (robot description, xacro)
@@ -9,5 +9,4 @@
     <xacro:property name='H' value='${dims["H"]}'/>
     <!-- wheel radius and length -->
-    <!-- <xacro:property name='R' value='${H}'/> -->
     <xacro:property name='R' value='${1.25*H}'/>
     <xacro:property name='WL' value='${W/5}'/>

File: diff_drive/urdf/ddrive.urdf.xacro (robot description, xacro)
@@ -10,14 +10,9 @@
     <xacro:property name='H' value='${dims["H"]}'/>
     <!-- wheel radius and length -->
-    <!-- <xacro:property name='R' value='${H}'/> -->
     <xacro:property name='R' value='${1.25*H}'/>
     <xacro:property name='WL' value='${W/5}'/>
     <!-- masses -->
-    <!-- <xacro:property name='MR' value='1'/> -->
     <xacro:property name='MW' value='0.5'/>
-    <!-- <xacro:property name='MC' value='0.5'/> -->
-    <!-- default for masses for rect -->
     <xacro:property name='MR' value='0.01'/>
-    <!-- <xacro:property name='MW' value='0.02'/> -->
     <xacro:property name='MC' value='0.01'/>
     <link name='base_footprint' type='fixed'/>
